Commit message: update

File: trans_mimic/robots/urdf/spot_arm/urdf/spot_arm.urdf (robot description, URDF)
Before this commit: robot spot, 21 links, 20 joints
Links:
- added link fl_toe; collision sphere radius=0.02; visual sphere radius=0.01
- added link fr_toe; collision sphere radius=0.02; visual sphere radius=0.01
- added link hl_toe; collision sphere radius=0.02; visual sphere radius=0.01
- added link hr_toe; collision sphere radius=0.02; visual sphere radius=0.01
Joints:
- added joint fl_toe_fixed: type fixed, parent fl.lleg, child fl_toe, origin xyz=0 0 -0.3205 rpy=0 0 0
- added joint fr_toe_fixed: type fixed, parent fr.lleg, child fr_toe, origin xyz=0 0 -0.3205 rpy=0 0 0
- added joint hl_toe_fixed: type fixed, parent hl.lleg, child hl_toe, origin xyz=0 0 -0.3205 rpy=0 0 0
- added joint hr_toe_fixed: type fixed, parent hr.lleg, child hr_toe, origin xyz=0 0 -0.3205 rpy=0 0 0
